Commit message: Add files via upload

File: rover_sim/urdf/rover_description.urdf (robot description, URDF)
Before this commit: robot rover_description, 26 links, 25 joints
Joints:
- joint body_rocker_left: type continuous -> revolute
- joint body_rocker_right: type continuous -> revolute

Commit message: Add files via upload

File: rover_sim/urdf/rover_description.urdf (robot description, URDF)
Before this commit: robot rover_description, 26 links, 25 joints
Joints:
- joint body_rocker_left: type revolute -> continuous
- joint body_rocker_right: type revolute -> continuous
